File: kicad/schematic.kicad_sch (KiCad schematic)
At the start: 7 parts, among them SW1 SW_Push, U1 ESP32-C3-WROOM-02, U2 ER_OLEDM0.91_1x-I2C

Commit message: improve schematics
Parts:
- RV1, RV2: value R_Potentiometer_Small -> 500k
Other:
- company: (none) -> FraI3mega
- title: (none) -> Temp-calc
Changed lines of the file:
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@@
 	(generator_version "10.0")
 	(paper "A4")
+	(title_block
+		(title "Temp-calc")
+		(date "2026-07-17")
+		(company "FraI3mega")
+		(comment 1 "Just a reference")
+	)
 	(junction
 		(at 120.65 104.14)
@@
 			)
 		)
-		(property "Value" "R_Potentiometer_Small"
+		(property "Value" "500k"
 			(at 107.95 97.79 90)
 			(show_name no)
@@
 			)
 		)
-		(property "Value" "R_Potentiometer_Small"
+		(property "Value" "500k"
 			(at 134.62 97.79 90)
 			(show_name no)
